Commit message: add tianracer_script to tianracer_navigation

File: tianracer_description/urdf/tianracer_compact.urdf (robot description, URDF)
Before this commit: robot tianracer_description, 12 links, 11 joints
Joints:
- joint laser_joint: origin xyz=0.22409 -0.0018403 0.1004 rpy=0 0 0 -> xyz=0.22409 -0.0018403 0.1004 rpy=0 0 3.1415926535
